Commit message: update

File: models/reBot-DevArm_description/urdf/reBot-DevArm.urdf (robot description, URDF)
Before this commit: robot reBot-DevArm, 8 links, 7 joints
Joints:
- joint joint2: axis 0 0 1 -> 0 0 -1; limit lower=0 upper=3.14 effort=27 velocity=50 -> lower=-3.14 upper=0 effort=27 velocity=50
- joint joint3: axis 0 0 -1 -> 0 0 1; limit lower=0 upper=3.14 effort=27 velocity=50 -> lower=-3.14 upper=0 effort=27 velocity=50
- joint joint4: axis 0 0 -1 -> 0 0 1
